Commit message: 提交1

File: src/car/model/car.urdf (robot description, URDF)
Before this commit: robot balance_car, 4 links, 3 joints
Links:
- added link left_front_lower_link, mass 0.12; collision cylinder length=0.3130 radius=0.011; visual cylinder length=0.3130 radius=0.011
- added link left_front_upper_link, mass 0.09; collision cylinder length=0.1844 radius=0.012; visual cylinder length=0.1844 radius=0.012
- added link left_rear_lower_link, mass 0.12; collision cylinder length=0.3130 radius=0.011; visual cylinder length=0.3130 radius=0.011
- added link left_rear_upper_link, mass 0.09; collision cylinder length=0.1844 radius=0.012; visual cylinder length=0.1844 radius=0.012
- added link left_wheel_carrier, mass 0.09; collision cylinder length=0.12 radius=0.025; visual cylinder length=0.12 radius=0.025
- added link right_front_lower_link, mass 0.12; collision cylinder length=0.3130 radius=0.011; visual cylinder length=0.3130 radius=0.011
- added link right_front_upper_link, mass 0.09; collision cylinder length=0.1844 radius=0.012; visual cylinder length=0.1844 radius=0.012
- added link right_rear_lower_link, mass 0.12; collision cylinder length=0.3130 radius=0.011; visual cylinder length=0.3130 radius=0.011
- added link right_rear_upper_link, mass 0.09; collision cylinder length=0.1844 radius=0.012; visual cylinder length=0.1844 radius=0.012
- added link right_wheel_carrier, mass 0.09; collision cylinder length=0.12 radius=0.025; visual cylinder length=0.12 radius=0.025
- link base_link: mass 1.0 -> 2.30; geometry collision box size=0.24 0.22 0.24; collision box size=0.38 0.36 0.12
- link left_wheel: mass 0.2 -> 0.32; geometry collision cylinder length=0.055 radius=0.10; visual cylinder length=0.055 radius=0.10
- link right_wheel: mass 0.2 -> 0.32; geometry collision cylinder length=0.055 radius=0.10; visual cylinder length=0.055 radius=0.10
Joints:
- added joint left_front_hip_joint: type revolute, parent base_link, child left_front_upper_link, origin xyz=0.14 0.17 0.36 rpy=0 0 0, axis 0 1 0, limit lower=-1.20 upper=1.20 effort=18 velocity=10
- added joint left_front_knee_joint: type revolute, parent left_front_upper_link, child left_front_lower_link, origin xyz=0.14 0 -0.12 rpy=0 0 0, axis 0 1 0, limit lower=-2.40 upper=2.40 effort=3 velocity=12
- added joint left_rear_ankle_joint: type revolute, parent left_rear_lower_link, child left_wheel_carrier, origin xyz=0.28 0 -0.14 rpy=0 0 0, axis 0 1 0, limit lower=-2.80 upper=2.80 effort=3 velocity=12
- added joint left_rear_hip_joint: type revolute, parent base_link, child left_rear_upper_link, origin xyz=-0.14 0.17 0.36 rpy=0 0 0, axis 0 1 0, limit lower=-1.20 upper=1.20 effort=18 velocity=10
- added joint left_rear_knee_joint: type revolute, parent left_rear_upper_link, child left_rear_lower_link, origin xyz=-0.14 0 -0.12 rpy=0 0 0, axis 0 1 0, limit lower=-2.40 upper=2.40 effort=3 velocity=12
- added joint right_front_hip_joint: type revolute, parent base_link, child right_front_upper_link, origin xyz=0.14 -0.17 0.36 rpy=0 0 0, axis 0 1 0, limit lower=-1.20 upper=1.20 effort=18 velocity=10
- added joint right_front_knee_joint: type revolute, parent right_front_upper_link, child right_front_lower_link, origin xyz=0.14 0 -0.12 rpy=0 0 0, axis 0 1 0, limit lower=-2.40 upper=2.40 effort=3 velocity=12
- added joint right_rear_ankle_joint: type revolute, parent right_rear_lower_link, child right_wheel_carrier, origin xyz=0.28 0 -0.14 rpy=0 0 0, axis 0 1 0, limit lower=-2.80 upper=2.80 effort=3 velocity=12
- added joint right_rear_hip_joint: type revolute, parent base_link, child right_rear_upper_link, origin xyz=-0.14 -0.17 0.36 rpy=0 0 0, axis 0 1 0, limit lower=-1.20 upper=1.20 effort=18 velocity=10
- added joint right_rear_knee_joint: type revolute, parent right_rear_upper_link, child right_rear_lower_link, origin xyz=-0.14 0 -0.12 rpy=0 0 0, axis 0 1 0, limit lower=-2.40 upper=2.40 effort=3 velocity=12
- joint left_wheel_joint: limit effort=10 velocity=10 -> effort=16 velocity=45; origin xyz=0 0.10 0.05 rpy=0 0 0 -> xyz=0 0.06 0 rpy=0 0 0; parent base_link -> left_wheel_carrier
- joint right_wheel_joint: limit effort=10 velocity=10 -> effort=16 velocity=45; origin xyz=0 -0.10 0.05 rpy=0 0 0 -> xyz=0 -0.06 0 rpy=0 0 0; parent base_link -> right_wheel_carrier

Commit message: 修正轮足机器人的URDF

File: src/car/model/car.urdf (robot description, URDF)
Before this commit: robot five_bar_wheel_leg_balance_car, 14 links, 13 joints
Joints:
- joint left_front_hip_joint: limit lower=-1.20 upper=1.20 effort=18 velocity=10 -> lower=0.1 upper=1.8 effort=18 velocity=10
- joint left_front_knee_joint: limit lower=-2.40 upper=2.40 effort=3 velocity=12 -> lower=0 upper=3.14159 effort=3 velocity=12; origin xyz=0.14 0 -0.12 rpy=0 0 0 -> xyz=0.1844 0 0 rpy=0 0 0
- joint left_rear_ankle_joint: origin xyz=0.28 0 -0.14 rpy=0 0 0 -> xyz=0.3130 0 0 rpy=0 0 0
- joint left_rear_hip_joint: limit lower=-1.20 upper=1.20 effort=18 velocity=10 -> lower=1.34159 upper=3.041592 effort=18 velocity=10
- joint left_rear_knee_joint: limit lower=-2.40 upper=2.40 effort=3 velocity=12 -> lower=-3.14159 upper=0 effort=3 velocity=12; origin xyz=-0.14 0 -0.12 rpy=0 0 0 -> xyz=0.1844 0 0 rpy=0 0 0
- joint right_front_hip_joint: limit lower=-1.20 upper=1.20 effort=18 velocity=10 -> lower=0.1 upper=1.8 effort=18 velocity=10
- joint right_front_knee_joint: limit lower=-2.40 upper=2.40 effort=3 velocity=12 -> lower=0 upper=3.14159 effort=3 velocity=12; origin xyz=0.14 0 -0.12 rpy=0 0 0 -> xyz=0.1844 0 0 rpy=0 0 0
- joint right_rear_ankle_joint: origin xyz=0.28 0 -0.14 rpy=0 0 0 -> xyz=0.3130 0 0 rpy=0 0 0
- joint right_rear_hip_joint: limit lower=-1.20 upper=1.20 effort=18 velocity=10 -> lower=1.34159 upper=3.041592 effort=18 velocity=10
- joint right_rear_knee_joint: limit lower=-2.40 upper=2.40 effort=3 velocity=12 -> lower=-3.14159 upper=0 effort=3 velocity=12; origin xyz=-0.14 0 -0.12 rpy=0 0 0 -> xyz=0.1844 0 0 rpy=0 0 0

Commit message: 1

File: src/car/model/car.urdf (robot description, URDF)
Before this commit: robot five_bar_wheel_leg_balance_car, 14 links, 13 joints
Joints:
- joint left_front_hip_joint: origin xyz=0.14 0.17 0.36 rpy=0 0 0 -> xyz=0.11 0.17 0.36 rpy=0 0 0
- joint left_rear_hip_joint: origin xyz=-0.14 0.17 0.36 rpy=0 0 0 -> xyz=-0.11 0.17 0.36 rpy=0 0 0
- joint right_front_hip_joint: origin xyz=0.14 -0.17 0.36 rpy=0 0 0 -> xyz=0.11 -0.17 0.36 rpy=0 0 0
- joint right_rear_hip_joint: origin xyz=-0.14 -0.17 0.36 rpy=0 0 0 -> xyz=-0.11 -0.17 0.36 rpy=0 0 0
