Commit message: 修正符号

File: src/car/model/car.urdf (robot description, URDF)
Before this commit: robot five_bar_wheel_leg_balance_car, 14 links, 13 joints
Joints:
- joint left_front_hip_joint: origin xyz=0.11 0.17 0.36 rpy=0 0 0 -> xyz=0.11 0.17 0 rpy=0 0 0
- joint left_rear_hip_joint: origin xyz=-0.11 0.17 0.36 rpy=0 0 0 -> xyz=-0.11 0.17 0 rpy=0 0 0
- joint right_front_hip_joint: origin xyz=0.11 -0.17 0.36 rpy=0 0 0 -> xyz=0.11 -0.17 0 rpy=0 0 0
- joint right_rear_hip_joint: origin xyz=-0.11 -0.17 0.36 rpy=0 0 0 -> xyz=-0.11 -0.17 0 rpy=0 0 0
